Commit message: env without goal reach cateria

File: jackal_envs/envs/assets/urdf/accessories.urdf.xacro (robot description, xacro)
@@ -18,5 +18,4 @@
       <xacro:include filename="$(env GAZEBO_ASSETS_PATH)/urdf/accessories/VLP-16.urdf.xacro" />
       <VLP-16 parent="$(optenv JACKAL_LASER_MOUNT front)_mount"
-              topic="$(optenv JACKAL_LASER_TOPIC front/scan)"
               name="front_laser">
         <origin xyz="0 0 0" rpy="0 0 0" />

File: jackal_envs/envs/assets/urdf/accessories/VLP-16.urdf.xacro (robot description, xacro)
@@ -2,5 +2,5 @@
 <robot xmlns:xacro="http://www.ros.org/wiki/xacro">
   <xacro:property name="M_PI" value="3.1415926535897931" />
-  <xacro:macro name="VLP-16" params="*origin parent:=base_link name:=velodyne topic:=/velodyne_points hz:=10 lasers:=16 samples:=1875 collision_range:=0.3 min_range:=0.9 max_range:=130.0 noise:=0.008 min_angle:=-${M_PI} max_angle:=${M_PI} gpu:=false">
+  <xacro:macro name="VLP-16" params="*origin parent:=base_link name:=velodyne topic:=/velodyne_points hz:=10 lasers:=16 samples:=1875 collision_range:=0.3 min_range:=0.2 max_range:=30.0 noise:=0.008 min_angle:=-${M_PI} max_angle:=${M_PI} gpu:=false">
     <joint name="${name}_base_mount_joint" type="fixed">
       <xacro:insert_block name="origin" />

File: jackal_envs/envs/assets/urdf/accessories/sick_lms1xx_mount.urdf.xacro (robot description, xacro)
@@ -34,5 +34,5 @@
         <geometry>
           <!-- Origin of this mesh is the base of the bracket. -->
-          <mesh filename="$(env GAZEBO_ASSETS_PATH)/meshes/sick-lms1xx-bracket.stl" />
+          <mesh filename="package://jackal_description/meshes/sick-lms1xx-bracket.stl" />
         </geometry>
         <material name="dark_grey" />

File: jackal_envs/envs/assets/urdf/jackal.urdf.xacro (robot description, xacro)
@@ -22,5 +22,5 @@
         <origin xyz="0 0 0" rpy="${PI/2} 0 0"/>
         <geometry>
-          <mesh filename="$(env GAZEBO_ASSETS_PATH)/meshes/jackal-wheel.stl"/>
+          <mesh filename="package://jackal_description/meshes/jackal-wheel.stl"/>
         </geometry>
         <material name="black" />
@@ -90,5 +90,5 @@
       <origin xyz="0 0 ${footprint_vertical_offset}" rpy="${PI/2} 0 ${PI/2}"/>
       <geometry>
-        <mesh filename="$(env GAZEBO_ASSETS_PATH)/meshes/jackal-base.stl"/>
+        <mesh filename="package://jackal_description/meshes/jackal-base.stl"/>
       </geometry>
       <material name="dark_grey" />
@@ -115,5 +115,5 @@
       <visual>
         <geometry>
-          <mesh filename="$(env GAZEBO_ASSETS_PATH)/meshes/jackal-fender.stl"/>
+          <mesh filename="package://jackal_description/meshes/jackal-fender.stl"/>
         </geometry>
         <material name="yellow" />
@@ -146,5 +146,5 @@
       <visual>
         <geometry>
-          <mesh filename="$(env GAZEBO_ASSETS_PATH)/meshes/jackal-fender.stl"/>
+          <mesh filename="package://jackal_description/meshes/jackal-fender.stl"/>
         </geometry>
         <material name="yellow" />
